File: ERDEM-İLİM/PCB çizimleri/PCB çizimleri.sch (KiCad schematic (older format))
At the start: 61 parts, among them Q1 BC547, Q2 BC547, Q3 BC547, Q4 BC547, U1 LM741, U10 IRFZ44N, U11 LM741, U12 IRFZ44N, U13 fan, U14 LM35-LP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

Commit message: .
.
Parts:
- gave numbers to parts that had none: 1
Changed lines of the file:
@@
 $EndComp
 $Comp
-L Erdem:röle U?
+L Erdem:röle U5
 U 1 1 60731FC1
 P 5200 2250
-F 0 "U?" H 5428 2321 50  0000 L CNN
+F 0 "U5" H 5428 2321 50  0000 L CNN
 F 1 "röle" H 5428 2230 50  0000 L CNN
 F 2 "" H 4900 2100 50  0001 C CNN
