File: PCB/electronic load/_autosave-electronic load.sch (KiCad schematic (older format))
At the start: 61 parts, among them J1 POWER, J2 LOAD_POSITIVE, J3 LOAD_NEGATIVE, M1 Fan, Q1 IRFZ46N, Q2 IRFZ46N, Q3 IRFZ46N, Q4 IRFZ46N, Q5 BC547, Q6 BC547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

Commit message: PCB-not complated
.
Parts:
- F1: footprint (none) -> erdem_lib:fuse
- J1, J2, J3: footprint (none) -> erdem_lib:klemens 2li
- RV1, RV2, RV3: footprint Resistor_THT:R_Axial_DIN0207_L6.3mm_D2.5mm_P7.62mm_Horizontal -> erdem_lib:pot
- SW1: footprint (none) -> Connector_PinHeader_2.00mm:PinHeader_1x03_P2.00mm_Horizontal
- U2, U3, U4, U5, U6, U7: footprint (none) -> Package_DIP:DIP-8_W7.62mm
Connections:
- net GND: no longer D2.2 (A), D3.2 (A), D4.2 (A), D5.2 (A), R4.2, R5.2, R6.2, R7.2
- net at Q1.3 (S), R12.1, U3.2 (-)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: now also D2.2 (A), R4.2
- net at Q2.3 (S), R13.1, U4.2 (-): now also D3.2 (A), R5.2
- net at Q3.3 (S), R14.1, U5.2 (-): now also D4.2 (A), R6.2
- net at Q4.3 (S), R15.1, U6.2 (-): now also D5.2 (A), R7.2
Other:
- moved on the sheet: C4, C5, C6, C7, R4, R5, R6, R7
