File: PCB/electronic load/electronic load.kicad_pcb (KiCad board)
At the start: 2 copper layers, 138.2 x 100.1 mm, 61 parts, among them J1 POWER, J2 LOAD_POSITIVE, J3 LOAD_NEGATIVE, M1 Fan, Q1 IRFZ46N, Q2 IRFZ46N, Q3 IRFZ46N, Q4 IRFZ46N, Q5 BC547, Q6 BC547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

Commit message: PCB- not finished
.
Parts:
- D2, D3, D4, D5: footprint Diode_THT:D_A-405_P10.16mm_Horizontal -> Diode_THT:D_A-405_P12.70mm_Horizontal
- F1, Q9: moved to B.Cu
- moved R17 176.0 mm to (122.2, 31.2), turned to 180 degrees
- moved R2 162.8 mm to (135.4, 60.2), turned to 270 degrees
- moved C3 157.0 mm to (138.9, 21.3), turned to 270 degrees
- moved R16 156.4 mm to (114.6, 34.8)
- moved R20 139.8 mm to (143.8, 27.9), turned to 180 degrees
- moved R3 137.0 mm to (143.8, 32.8), turned to 180 degrees
- moved R22 136.1 mm to (143.8, 43.9), turned to 180 degrees
- moved R18 130.5 mm to (136.1, 36.3)
- moved R21 127.2 mm to (143.8, 40.1), turned to 180 degrees
- moved U2 115.2 mm to (120.1, 67.8), turned to 90 degrees
- moved R19 105.7 mm to (137.9, 56.4), turned to 180 degrees
- moved R1 95.7 mm to (131.6, 67.8), turned to 90 degrees
- moved R13 38.2 mm to (53.6, 16.5), turned to 270 degrees
- moved C4 35.0 mm to (65.0, 33.3)
- moved R12 33.5 mm to (98.0, 16.5), turned to 270 degrees
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Connections:
- U2 pad 4: Net-(U2-Pad4) -> GND
- U7 pad 4: Net-(U7-Pad4) -> GND
Routing:
- net GND: track 0.00 -> 450.1 mm, vias 0 -> 3
- net V_DRAIN: track 0.00 -> 316.6 mm
- net IREF: track 0.00 -> 99.6 mm, vias 0 -> 3
- net 12V: track 0.00 -> 80.5 mm, vias 0 -> 3
- net Net-(D2-Pad2): track 0.00 -> 72.9 mm
- net Net-(D4-Pad2): track 0.00 -> 45.5 mm
- net Net-(D5-Pad2): track 0.00 -> 45.4 mm
- net Net-(D3-Pad2): track 0.00 -> 45.2 mm
- net Net-(D7-Pad2): track 0.00 -> 29.2 mm, vias 0 -> 2
- net Net-(C5-Pad1): track 0.00 -> 24.0 mm
- net Net-(C7-Pad1): track 0.00 -> 22.5 mm
- net Net-(C4-Pad1): track 0.00 -> 22.0 mm
- net Net-(C6-Pad1): track 0.00 -> 21.7 mm
- net Net-(RV2-Pad2): track 0.00 -> 21.4 mm
- net Net-(RV1-Pad2): track 0.00 -> 21.2 mm
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Other:
- board size 138.2 x 100.1 mm -> 138.2 x 100.3 mm

Commit message: PCB finished
.
Parts:
- U1: footprint Package_TO_SOT_THT:TO-92_Inline -> Package_TO_SOT_THT:TO-92_Inline_Wide
- moved U1 13.6 mm to (125.0, 36.1), turned to 0 degrees
- moved C1 7.89 mm to (123.7, 41.7), turned to 0 degrees
- moved C2 7.37 mm to (131.6, 41.7), turned to 180 degrees
- moved R2 3.06 mm to (135.1, 57.1)
- moved R1 3.06 mm to (131.3, 64.8)
- moved U2 3.06 mm to (119.9, 64.8)
- moved R19 3.06 mm to (137.7, 53.3)
Routing:
- net GND: track 450.1 -> 916.2 mm, vias 3 -> 10
- net 12V: track 80.5 -> 444.6 mm, vias 3 -> 14
- net HALT: track 0.00 -> 285.3 mm, vias 0 -> 10
- net IREF: track 99.6 -> 357.9 mm, vias 3 -> 8
- net Net-(D1-Pad2): track 0.00 -> 47.7 mm, vias 0 -> 2
- net Net-(C6-Pad1): track 21.7 -> 48.1 mm
- net 3.3V: track 4.34 -> 28.1 mm
- net Net-(C7-Pad1): track 22.5 -> 45.2 mm
- net Net-(C5-Pad1): track 24.0 -> 45.8 mm
- net Net-(C4-Pad1): track 22.0 -> 43.0 mm
- net Net-(D5-Pad2): track 45.4 -> 55.4 mm
- net Net-(D2-Pad2): track 72.9 -> 82.5 mm
- net Net-(R1-Pad1): track 3.81 -> 13.2 mm
- net Net-(D7-Pad2): track 29.2 -> 36.9 mm
- net Net-(D4-Pad2): track 45.5 -> 49.9 mm
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- added copper zone on B.Cu, net GND
- added copper zone on B.Cu, net Net-(F1-Pad1)
- added copper zone on B.Cu, net V_DRAIN
Other:
- outline, holes or cut-outs redrawn
