File: PCB/electronic load/electronic load.sch (KiCad schematic (older format))
At the start: 62 parts, among them J1 POWER, J2 LOAD_POSITIVE, J3 LOAD_NEGATIVE, M1 Fan, M2 Fan, Q1 IRFZ46N, Q2 IRFZ46N, Q3 IRFZ46N, Q4 IRFZ46N, Q5 BC547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

Commit message: PCB-not complated
.
Parts:
- removed M2: Fan, symbol Motor:Fan
- C1, C2, C3, C4, C5, C6, C7: footprint (none) -> Capacitor_THT:CP_Radial_D5.0mm_P2.00mm
- D1, D6, D7: footprint (none) -> LED_THT:LED_D3.0mm_FlatTop
- D2, D3, D4, D5: footprint (none) -> Diode_THT:D_A-405_P10.16mm_Horizontal
- F1: footprint (none) -> erdem_lib:fuse
- J1, J2, J3: footprint (none) -> erdem_lib:klemens 2li
- M1: footprint (none) -> Connector_PinHeader_2.00mm:PinHeader_1x02_P2.00mm_Vertical
- Q1, Q2, Q3, Q4: footprint (none) -> Package_TO_SOT_THT:TO-220-3_Horizontal_TabUp
- Q5, Q6, Q7, Q8: footprint (none) -> Package_TO_SOT_THT:TO-92_Inline_Wide
- Q9: footprint (none) -> Package_TO_SOT_SMD:SOT-23
- R1, R10, R11, R16, R17, R18, R19, R2, R20, R21, R22, R3, R4, R5, R6, R7, R8, R9, RV1, RV2, RV3: footprint (none) -> Resistor_THT:R_Axial_DIN0207_L6.3mm_D2.5mm_P7.62mm_Horizontal
- R12, R13, R14, R15: footprint (none) -> Resistor_THT:R_Axial_Power_L25.0mm_W9.0mm_P27.94mm
- SW1: footprint (none) -> Connector_PinHeader_2.00mm:PinHeader_1x03_P2.00mm_Horizontal
- U2, U3, U4, U5, U6, U7: footprint (none) -> Package_DIP:DIP-8_W7.62mm
Other:
- moved on the sheet: M1

Commit message: PCB- not finished
.
Parts:
- D2, D3, D4, D5: footprint Diode_THT:D_A-405_P10.16mm_Horizontal -> Diode_THT:D_A-405_P12.70mm_Horizontal
- RV1, RV2, RV3: footprint Resistor_THT:R_Axial_DIN0207_L6.3mm_D2.5mm_P7.62mm_Horizontal -> erdem_lib:pot
Connections:
- net GND: now also U2.4 (V-), U7.4 (V-); no longer D2.2 (A), D3.2 (A), D4.2 (A), D5.2 (A), R4.2, R5.2, R6.2, R7.2
- net at Q1.3 (S), R12.1, U3.2 (-)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: now also D2.2 (A), R4.2
- net at Q2.3 (S), R13.1, U4.2 (-): now also D3.2 (A), R5.2
- net at Q3.3 (S), R14.1, U5.2 (-): now also D4.2 (A), R6.2
- net at Q4.3 (S), R15.1, U6.2 (-): now also D5.2 (A), R7.2
Other:
- moved on the sheet: C4, C5, C6, C7, R4, R5, R6, R7

Commit message: PCB finished
.
Parts:
- U1: footprint Package_TO_SOT_THT:TO-92_Inline -> Package_TO_SOT_THT:TO-92_Inline_Wide
Changed lines of the file:
@@
 F 0 "U1" H 10800 1942 50  0000 C CNN
 F 1 "L78L33_TO92" H 10800 1851 50  0000 C CNN
-F 2 "Package_TO_SOT_THT:TO-92_Inline" H 10800 1925 50  0001 C CIN
+F 2 "Package_TO_SOT_THT:TO-92_Inline_Wide" H 10800 1925 50  0001 C CIN
 F 3 "http://www.st.com/content/ccc/resource/technical/document/datasheet/15/55/e5/aa/23/5b/43/fd/CD00000446.pdf/files/CD00000446.pdf/jcr:content/translations/en.CD00000446.pdf" H 10800 1650 50  0001 C CNN
 	1    10800 1700
